Commit message: Included OpenCV for ImageProcessor. Updated mesh and texture files

File: project/urdf/camera_description.urdf.xacro (robot description, xacro)
@@ -9,5 +9,5 @@
     <parent link="world"/>
     <child link="camera_link"/>
-    <origin xyz="1.9 0.25 1.675" rpy="0.0 ${pi/2.6} ${pi}" />
+    <origin xyz="1.9 0.25 1.2" rpy="0.0 ${pi/2.6} ${pi}" />
   </joint>
   <!-- Link camera with world joint -->

File: project/urdf/robot_description.urdf.xacro (robot description, xacro)
@@ -6,10 +6,10 @@
   <xacro:include filename="$(find ur_description)/urdf/ur5e.xacro" />
   <!-- <xacro:ur5e_robot prefix="" /> -->
-  <link name="world" />
+  <!-- <link name="world" />
   <joint name="world_to_base" type="fixed">
     <parent link="world"/>
     <child link="base_link"/>
     <origin xyz="0.8 0.0 0.675" rpy="0.0 0.0 0.0" />
-  </joint>
+  </joint>  -->
   <!-- Link robot with world joint -->
   <!-- TODO: INSERT CODE HERE -->

Commit message: Updated URDF and models to contain Lab09 E-pick functionality

File: project/urdf/camera_description.urdf.xacro (robot description, xacro)
@@ -1,15 +1,12 @@
 <?xml version="1.0"?>
-<robot xmlns:xacro="http://ros.org/wiki/xacro"
-       name="camera" >
-  <!-- Include camera description (Hint: look at camera_model.urdf.xacro within the lab08_activity package) -->
-  <!-- TODO: INSERT CODE HERE -->
-  <xacro:include filename="$(find project)/urdf/camera_model.xacro"/>
+<robot xmlns:xacro="http://ros.org/wiki/xacro" name="camera" >
+  <!-- Include camera description -->
+  <xacro:include filename="$(find project)/urdf/inc/camera_model.xacro" />
   <link name="world" />
-  <joint name="camera_joint" type="fixed">
-    <parent link="world"/>
-    <child link="camera_link"/>
-    <origin xyz="1.9 0.25 1.2" rpy="0.0 ${pi/2.6} ${pi}" />
+  <!-- Link camera with world joint -->
+  <joint name="camera_world_joint" type="fixed">
+    <parent link="world" />
+    <child link = "camera_link" />
+    <origin xyz="1.9 0.25 1.675" rpy="0.0 ${pi/2.6} ${pi}" />
   </joint>
-  <!-- Link camera with world joint -->
-  <!-- TODO: INSERT CODE HERE -->
 </robot>

Commit message: Implemented User Move Spawning and Robot Move Service for Gazebo Controller

File: project/urdf/camera_description.urdf.xacro (robot description, xacro)
@@ -8,5 +8,5 @@
     <parent link="world" />
     <child link = "camera_link" />
-    <origin xyz="1.9 0.25 1.675" rpy="0.0 ${pi/2.6} ${pi}" />
+    <origin xyz="1.6 0.25 1.575" rpy="0.0 ${pi/2.6} ${pi}" />
   </joint>
 </robot>
